File: ESP-07/ESP-07.brd (EAGLE design)
At the start: 20.6 x 36.8 mm, 7 parts

Commit message: tweak layout
Routing:
- net N$6: track 20.2 -> 19.7 mm
Changed lines of the file:
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@@
 <?xml version="1.0" encoding="utf-8"?>
 <!DOCTYPE eagle SYSTEM "eagle.dtd">
-<eagle version="7.7.0">
+<eagle version="7.5.0">
 <drawing>
 <settings>
@@
 <setting verticaltext="up"/>
 </settings>
-<grid distance="0.05" unitdist="inch" unit="inch" style="lines" multiple="1" display="no" altdistance="0.025" altunitdist="inch" altunit="inch"/>
+<grid distance="0.01" unitdist="inch" unit="inch" style="lines" multiple="1" display="no" altdistance="0.025" altunitdist="inch" altunit="inch"/>
 <layers>
 <layer number="1" name="Top" color="4" fill="1" visible="yes" active="yes"/>
@@
 <wire x1="19.05" y1="11.75" x2="20.32" y2="10.48" width="0.4064" layer="1"/>
 <wire x1="20.32" y1="10.48" x2="20.32" y2="8.89" width="0.4064" layer="1"/>
-<wire x1="19.05" y1="11.75" x2="17.145" y2="13.655" width="0.4064" layer="1"/>
-<wire x1="17.145" y1="13.655" x2="17.145" y2="24.765" width="0.4064" layer="1"/>
-<wire x1="17.145" y1="24.765" x2="18.12" y2="25.74" width="0.4064" layer="1"/>
-<wire x1="18.12" y1="25.74" x2="23.44" y2="25.74" width="0.4064" layer="1"/>
+<wire x1="19.05" y1="11.75" x2="17.399" y2="13.401" width="0.4064" layer="1"/>
+<wire x1="17.399" y1="13.401" x2="17.399" y2="24.765" width="0.4064" layer="1"/>
+<wire x1="17.399" y1="24.765" x2="18.374" y2="25.74" width="0.4064" layer="1"/>
+<wire x1="18.374" y1="25.74" x2="23.44" y2="25.74" width="0.4064" layer="1"/>
 </signal>
 <signal name="N$4">
@@
 <contactref element="R2" pad="1"/>
 <contactref element="U$1" pad="CH_PD"/>
-<wire x1="14.285" y1="16.51" x2="14.605" y2="16.825" width="0.4064" layer="1"/>
-<wire x1="14.605" y1="16.825" x2="14.605" y2="28.575" width="0.4064" layer="1"/>
-<wire x1="14.605" y1="28.575" x2="13.44" y2="29.74" width="0.4064" layer="1"/>
-<wire x1="13.44" y1="29.74" x2="7.04" y2="29.74" width="0.4064" layer="1"/>
+<wire x1="14.285" y1="16.51" x2="14.097" y2="16.825" width="0.4064" layer="1"/>
+<wire x1="14.097" y1="16.825" x2="14.097" y2="28.575" width="0.4064" layer="1"/>
+<wire x1="14.097" y1="28.575" x2="12.932" y2="29.74" width="0.4064" layer="1"/>
+<wire x1="12.932" y1="29.74" x2="7.04" y2="29.74" width="0.4064" layer="1"/>
 </signal>
 <signal name="N$2">
 <contactref element="U$1" pad="TX"/>
 <contactref element="SV1" pad="3"/>
-<wire x1="12.7" y1="8.89" x2="15.875" y2="12.065" width="0.4064" layer="1"/>
-<wire x1="15.875" y1="12.065" x2="15.875" y2="32.385" width="0.4064" layer="1"/>
-<wire x1="15.875" y1="32.385" x2="17.23" y2="33.74" width="0.4064" layer="1"/>
+<wire x1="12.7" y1="8.89" x2="15.621" y2="11.811" width="0.4064" layer="1"/>
+<wire x1="15.621" y1="11.811" x2="15.621" y2="32.385" width="0.4064" layer="1"/>
+<wire x1="15.621" y1="32.385" x2="17.23" y2="33.74" width="0.4064" layer="1"/>
 <wire x1="17.23" y1="33.74" x2="23.44" y2="33.74" width="0.4064" layer="1"/>
 </signal>
@@
 <wire x1="15.24" y1="8.89" x2="16.51" y2="10.16" width="0.4064" layer="1"/>
 <wire x1="16.51" y1="10.16" x2="16.51" y2="30.48" width="0.4064" layer="1"/>
-<wire x1="16.51" y1="30.48" x2="17.77" y2="31.74" width="0.4064" layer="1"/>
-<wire x1="17.77" y1="31.74" x2="23.44" y2="31.74" width="0.4064" layer="1"/>
+<wire x1="16.51" y1="30.48" x2="18.024" y2="31.74" width="0.4064" layer="1"/>
+<wire x1="18.024" y1="31.74" x2="23.44" y2="31.74" width="0.4064" layer="1"/>
 </signal>
 </signals>
